File: images/kicad/electric-circuits/electric-circuits_02.kicad_sch (KiCad schematic)
At the start: 44 parts

Commit message: 22/01/2025 Update
Parts:
- removed V? (x5): 2V, symbol electric-circuits-rescue:Pila-simbolos
- added V3, V4, V5, V6, V7: 2V, symbol electric-circuits-rescue:Pila-simbolos
Connections:
- net at R1., V?.: now also S1.; no longer R2.
- net at V?.: now also R2.; no longer R1.
- net at R2.: now also R1.; no longer V?.
- net at R?., R?.: now also R?. (x2)
- net at R2., R3., V?.: now also S1.; no longer R1.
- net at D1., D2., D3.: no longer D4., V?.
- net at D?., S2.: now also V?.; no longer R?.
- net at V?.: now also R1.; no longer S1.
- net at R1.: now also S2.; no longer V?.
- net at V?.: now also V3., V4.
- new net: R1., R2., V?. (x2)
- new net: R?., R?. (x3)
- new net: R1., V?.
- new net: R1., R2., R3., V?.
- new net: D1., D2., D3., D4., V?.
- new net: D?., R?., S2.
- new net: S1., V?.
- new net: V3., V4., V?.
- new net: V5., V6.
- new net: V6., V7.
- now unconnected: R?., R?.
