File: images/kicad/electric-circuits/electric-circuits_03.kicad_sch (KiCad schematic)
At the start: 38 parts

Commit message: 22/01/2025 Update
Connections:
- net at R?.: now also R?. (x2)
- net at R?.: now also R?.; no longer R?. (x2)
- net at R?.: no longer R?. (x2)
- net at V1.: now also V2.
- net at V2.: no longer V1.
- net at R?., R?.: now also R?., R?.
- net at R?., R?.: no longer R?., R?.
- net at L2., V?.: no longer L1.
- net at D1., D2.: now also D3., D4.; no longer V?.
- net at D5., D6.: now also D3., D4.; no longer V?.
- new net: R?., R?., R?. (x2)
- new net: R?., R?.
- new net: R1., R2., R3., V?.
- new net: L1., L2., V?.
- new net: D1., D2., V?.
- new net: D5., D6., V?.
Changed lines of the file:
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@@
 		)
 	)
+	(wire
+		(pts
+			(xy 53.34 277.495) (xy 53.34 280.035)
+		)
+		(stroke
+			(width 0)
+			(type default)
+		)
+	)
 	(polyline
 		(pts
@@
 	(wire
 		(pts
+			(xy 53.34 254.635) (xy 53.34 257.175)
+		)
+		(stroke
+			(width 0)
+			(type default)
+		)
+	)
+	(wire
+		(pts
 			(xy 146.685 83.185) (xy 146.685 85.725)
 		)
@@
 			)
 		)
-		(pin "~"
+		(pin ""
 		)
-		(pin "~"
+		(pin ""
 		)
 	)
@@
 			)
 		)
-		(pin "~"
+		(pin ""
 		)
-		(pin "~"
+		(pin ""
 		)
 	)
@@
 			)
 		)
-		(pin "~"
+		(pin ""
 		)
-		(pin "~"
+		(pin ""
 		)
 	)
@@
 			)
 		)
-		(pin "~"
+		(pin ""
 		)
-		(pin "~"
+		(pin ""
 		)
 	)
@@
 			)
 		)
-		(pin "~"
+		(pin ""
 		)
-		(pin "~"
+		(pin ""
 		)
 	)
@@
 			)
 		)
-		(pin "~"
+		(pin ""
 		)
-		(pin "~"
+		(pin ""
 		)
 	)
@@
 			)
 		)
-		(pin "~"
+		(pin ""
 		)
-		(pin "~"
+		(pin ""
 		)
 	)
@@
 			)
 		)
-		(pin "~"
+		(pin ""
 		)
-		(pin "~"
+		(pin ""
 		)
 	)
@@
 			)
 		)
-		(pin "~"
+		(pin ""
 		)
-		(pin "~"
+		(pin ""
 		)
 	)
@@
 			)
 		)
-		(pin "~"
+		(pin ""
 		)
-		(pin "~"
+		(pin ""
 		)
 	)
@@
 			)
 		)
-		(pin "~"
+		(pin ""
 		)
-		(pin "~"
+		(pin ""
 		)
 	)
@@
 			)
 		)
-		(pin "~"
+		(pin ""
 		)
-		(pin "~"
+		(pin ""
 		)
 	)
@@
 			)
 		)
-		(pin "~"
+		(pin ""
 		)
-		(pin "~"
+		(pin ""
 		)
 	)
@@
 			)
 		)
-		(pin "~"
+		(pin ""
 		)
-		(pin "~"
+		(pin ""
 		)
 	)
@@
 			)
 		)
-		(pin "~"
+		(pin ""
 		)
-		(pin "~"
+		(pin ""
 		)
 	)
@@
 			)
 		)
-		(pin "~"
+		(pin ""
 		)
-		(pin "~"
+		(pin ""
 		)
 	)
@@
 			)
 		)
-		(pin "~"
+		(pin ""
 		)
-		(pin "~"
+		(pin ""
 		)
 	)
@@
 			)
 		)
-		(pin "~"
+		(pin ""
 		)
-		(pin "~"
+		(pin ""
 		)
 	)
@@
 			)
 		)
-		(pin "~"
+		(pin ""
 		)
-		(pin "~"
+		(pin ""
 		)
 	)
@@
 			)
 		)
-		(pin "~"
+		(pin ""
 		)
-		(pin "~"
+		(pin ""
 		)
 	)
@@
 			)
 		)
-		(pin "~"
+		(pin ""
 		)
-		(pin "~"
+		(pin ""
 		)
 	)
@@
 			)
 		)
-		(pin "~"
+		(pin ""
 		)
-		(pin "~"
+		(pin ""
 		)
 	)
@@
 			)
 		)
-		(pin "~"
+		(pin ""
 		)
-		(pin "~"
+		(pin ""
 		)
 	)
@@
 			)
 		)
-		(pin "~"
+		(pin ""
 		)
-		(pin "~"
+		(pin ""
 		)
 	)
@@
 			)
 		)
-		(pin "~"
+		(pin ""
 		)
-		(pin "~"
+		(pin ""
 		)
 	)
@@
 			)
 		)
-		(pin "~"
+		(pin ""
 		)
-		(pin "~"
+		(pin ""
 		)
 	)
@@
 			)
 		)
-		(pin "~"
+		(pin ""
 		)
-		(pin "~"
+		(pin ""
 		)
 	)
@@
 			)
 		)
-		(pin "~"
+		(pin ""
 		)
-		(pin "~"
+		(pin ""
 		)
 	)
@@
 			)
 		)
-		(pin "~"
+		(pin ""
 		)
-		(pin "~"
+		(pin ""
 		)
 	)
@@
 			)
 		)
-		(pin "~"
+		(pin ""
 		)
-		(pin "~"
+		(pin ""
 		)
 	)
@@
 			)
 		)
-		(pin "~"
+		(pin ""
 		)
-		(pin "~"
+		(pin ""
 		)
 	)
@@
 			)
 		)
-		(pin "~"
+		(pin ""
 		)
-		(pin "~"
+		(pin ""
 		)
 	)
@@
 			)
 		)
-		(pin "~"
+		(pin ""
 		)
-		(pin "~"
+		(pin ""
 		)
 	)
@@
 			)
 		)
-		(pin "~"
+		(pin ""
 		)
-		(pin "~"
+		(pin ""
 		)
 	)
@@
 			)
 		)
-		(pin "~"
+		(pin ""
 		)
-		(pin "~"
+		(pin ""
 		)
 	)
@@
 			)
 		)
-		(pin "~"
+		(pin ""
 		)
-		(pin "~"
+		(pin ""
 		)
 	)
@@
 			)
 		)
-		(pin "~"
+		(pin ""
 		)
-		(pin "~"
+		(pin ""
 		)
 	)
