File: images/kicad/electric-digital/electric-digital.kicad_sch (KiCad schematic)
At the start: 67 parts, among them Q1 NPN, Q2 NPN, Q3 NPN, Q4 NPN, Q5 NPN, Q6 NPN, Q7 NPN, Q8 NPN, Q9 NPN

Commit message: 22/01/2025 Update
Parts:
- removed U? (x17): logic_nand, symbol electric-digital-rescue:logic_nand-simbolos
- added U1, U10, U11, U12, U13, U14, U15, U16, U17, U2, U3, U4, U5, U6, U7, U8, U9: logic_nand, symbol electric-digital-rescue:logic_nand-simbolos
Connections:
- net at Q8., Q9.: now also R?., o?.; no longer o?.
- net at U?. (B): now also U1. (B)
- net at U?. (B): now also U7. (B)
- new net: Q8., Q9., o?.
- new net: U6. (B), U?. (B)
- new net: U6. (B), U7. (B), U?. (B)
- new net: U13. (B), U15. (B)
- new net: U13. (B), U14. (B)
- new net: U4. (B), U5. (B)
- new net: U2. (B), U4. (B)
- new net: U3. (B), U4. (B)
- new net: U17. (B), U8. (B)
- new net: U6. (B), U8. (B)
- new net: U11. (B), U12. (B)
- new net: U11. (B), U9. (B)
- new net: U10. (B), U11. (B), U9. (B)
- new net: U10. (B), U12. (B)
- new net: U10. (B), U9. (B)
- new net: U7. (B), U8. (B)

Commit message: 29/07/2025 Update
Parts:
- U1, U10, U11, U12, U13, U14, U15, U16, U17, U2, U3, U4, U5, U6, U7, U8, U9, U? (x2): symbol electric-digital-rescue:logic_nand-simbolos -> simbolos-electricos:logic_nand
Connections:
- net at Q8., Q9.: now also R?., o?.; no longer o?.
- net at U?.: now also U1.
- net at U1.: no longer U?. (B)
- net at U?.: now also U7.; no longer U6. (B)
- net at U7.: now also U8.; no longer U?. (B)
- net at U13.: now also U14.
- net at U15.: no longer U13. (B)
- net at U14.: no longer U13. (B)
- net at U5.: now also U4.
- net at U4.: now also U3.; no longer U5. (B)
- net at U2.: now also U4.
- net at U3.: no longer U4. (B)
- net at U17.: now also U8.
- net at U11.: now also U10., U9.; no longer U12. (B)
- net at U9.: now also U10.; no longer U11. (B)
- net at U12.: now also U10.
- new net: Q8., Q9., o?.
- new net: U6., U?.
- new net: U6., U7., U?.
- new net: U13., U15.
- new net: U11., U12.
- new net: U11., U9.
Changed lines of the file:
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@@
 	)
 	(symbol
-		(lib_name "logic_nand-simbolos_1")
-		(lib_id "electric-digital-rescue:logic_nand-simbolos")
+		(lib_name "simbolos-electricos:logic_nand")
+		(lib_id "simbolos-electricos:logic_nand")
 		(at 38.1 264.16 0)
 		(unit 1)
@@
 	)
 	(symbol
-		(lib_name "logic_nand-simbolos_2")
-		(lib_id "electric-digital-rescue:logic_nand-simbolos")
+		(lib_name "simbolos-electricos:logic_nand")
+		(lib_id "simbolos-electricos:logic_nand")
 		(at 120.65 170.18 0)
 		(unit 1)
@@
 	)
 	(symbol
+		(lib_name "simbolos-electricos:NPN")
 		(lib_id "simbolos-electricos:NPN")
 		(at 66.675 173.355 0)
@@
 	)
 	(symbol
-		(lib_name "logic_nand-simbolos_1")
-		(lib_id "electric-digital-rescue:logic_nand-simbolos")
+		(lib_name "simbolos-electricos:logic_nand")
+		(lib_id "simbolos-electricos:logic_nand")
 		(at 163.83 74.93 0)
 		(unit 1)
@@
 	)
 	(symbol
+		(lib_name "simbolos-electricos:NPN")
 		(lib_id "simbolos-electricos:NPN")
 		(at 50.8 130.81 0)
@@
 	)
 	(symbol
-		(lib_name "logic_nand-simbolos_1")
-		(lib_id "electric-digital-rescue:logic_nand-simbolos")
+		(lib_name "simbolos-electricos:logic_nand")
+		(lib_id "simbolos-electricos:logic_nand")
 		(at 166.37 217.805 0)
 		(unit 1)
@@
 	)
 	(symbol
-		(lib_name "logic_nand-simbolos_1")
-		(lib_id "electric-digital-rescue:logic_nand-simbolos")
+		(lib_name "simbolos-electricos:logic_nand")
+		(lib_id "simbolos-electricos:logic_nand")
 		(at 127 210.185 0)
 		(unit 1)
@@
 	)
 	(symbol
-		(lib_name "logic_nand-simbolos_1")
-		(lib_id "electric-digital-rescue:logic_nand-simbolos")
+		(lib_name "simbolos-electricos:logic_nand")
+		(lib_id "simbolos-electricos:logic_nand")
 		(at 146.685 217.805 0)
 		(unit 1)
@@
 	)
 	(symbol
+		(lib_name "simbolos-electricos:NPN")
 		(lib_id "simbolos-electricos:NPN")
 		(at 67.31 67.31 0)
@@
 	)
 	(symbol
-		(lib_name "logic_nand-simbolos_1")
-		(lib_id "electric-digital-rescue:logic_nand-simbolos")
+		(lib_name "simbolos-electricos:logic_nand")
+		(lib_id "simbolos-electricos:logic_nand")
 		(at 139.065 67.31 0)
 		(unit 1)
@@
 	)
 	(symbol
+		(lib_name "simbolos-electricos:NPN")
 		(lib_id "simbolos-electricos:NPN")
 		(at 48.895 220.98 0)
@@
 	)
 	(symbol
+		(lib_name "simbolos-electricos:NPN")
 		(lib_id "simbolos-electricos:NPN")
 		(at 31.75 66.675 0)
@@
 	)
 	(symbol
+		(lib_name "simbolos-electricos:NPN")
 		(lib_id "simbolos-electricos:NPN")
 		(at 31.115 172.72 0)
@@
 	)
 	(symbol
-		(lib_name "logic_nand-simbolos_1")
-		(lib_id "electric-digital-rescue:logic_nand-simbolos")
+		(lib_name "simbolos-electricos:logic_nand")
+		(lib_id "simbolos-electricos:logic_nand")
 		(at 63.5 264.16 0)
 		(unit 1)
@@
 	)
 	(symbol
-		(lib_name "logic_nand-simbolos_1")
-		(lib_id "electric-digital-rescue:logic_nand-simbolos")
+		(lib_name "simbolos-electricos:logic_nand")
+		(lib_id "simbolos-electricos:logic_nand")
 		(at 172.085 170.18 0)
 		(unit 1)
@@
 	)
 	(symbol
-		(lib_name "logic_nand-simbolos_1")
-		(lib_id "electric-digital-rescue:logic_nand-simbolos")
+		(lib_name "simbolos-electricos:logic_nand")
+		(lib_id "simbolos-electricos:logic_nand")
 		(at 139.065 162.56 0)
 		(unit 1)
@@
 	)
 	(symbol
-		(lib_name "logic_nand-simbolos_1")
-		(lib_id "electric-digital-rescue:logic_nand-simbolos")
+		(lib_name "simbolos-electricos:logic_nand")
+		(lib_id "simbolos-electricos:logic_nand")
 		(at 152.4 128.27 0)
 		(unit 1)
@@
 	)
 	(symbol
-		(lib_name "logic_nand-simbolos_1")
-		(lib_id "electric-digital-rescue:logic_nand-simbolos")
+		(lib_name "simbolos-electricos:logic_nand")
+		(lib_id "simbolos-electricos:logic_nand")
 		(at 167.64 120.65 0)
 		(unit 1)
@@
 	)
 	(symbol
+		(lib_name "simbolos-electricos:NPN")
 		(lib_id "simbolos-electricos:NPN")
 		(at 50.8 120.65 0)
@@
 	)
 	(symbol
-		(lib_name "logic_nand-simbolos_1")
-		(lib_id "electric-digital-rescue:logic_nand-simbolos")
+		(lib_name "simbolos-electricos:logic_nand")
+		(lib_id "simbolos-electricos:logic_nand")
 		(at 130.81 120.65 0)
 		(unit 1)
@@
 	)
 	(symbol
-		(lib_name "logic_nand-simbolos_1")
-		(lib_id "electric-digital-rescue:logic_nand-simbolos")
+		(lib_name "simbolos-electricos:logic_nand")
+		(lib_id "simbolos-electricos:logic_nand")
 		(at 127 225.425 0)
 		(unit 1)
@@
 	)
 	(symbol
-		(lib_name "logic_nand-simbolos_1")
-		(lib_id "electric-digital-rescue:logic_nand-simbolos")
+		(lib_name "simbolos-electricos:logic_nand")
+		(lib_id "simbolos-electricos:logic_nand")
 		(at 154.305 170.18 0)
 		(unit 1)
@@
 	)
 	(symbol
-		(lib_name "logic_nand-simbolos_1")
-		(lib_id "electric-digital-rescue:logic_nand-simbolos")
+		(lib_name "simbolos-electricos:logic_nand")
+		(lib_id "simbolos-electricos:logic_nand")
 		(at 139.065 82.55 0)
 		(unit 1)
@@
 	)
 	(symbol
+		(lib_name "simbolos-electricos:NPN")
 		(lib_id "simbolos-electricos:NPN")
 		(at 50.8 24.13 0)
@@
 	)
 	(symbol
-		(lib_name "logic_nand-simbolos_1")
-		(lib_id "electric-digital-rescue:logic_nand-simbolos")
+		(lib_name "simbolos-electricos:logic_nand")
+		(lib_id "simbolos-electricos:logic_nand")
 		(at 152.4 113.03 0)
 		(unit 1)
@@
 	)
 	(symbol
-		(lib_name "logic_nand-simbolos_1")
-		(lib_id "electric-digital-rescue:logic_nand-simbolos")
+		(lib_name "simbolos-electricos:logic_nand")
+		(lib_id "simbolos-electricos:logic_nand")
 		(at 139.065 177.8 0)
 		(unit 1)
@@
 	)
 	(symbol
-		(lib_name "logic_nand-simbolos_1")
-		(lib_id "electric-digital-rescue:logic_nand-simbolos")
+		(lib_name "simbolos-electricos:logic_nand")
+		(lib_id "simbolos-electricos:logic_nand")
 		(at 148.59 26.035 0)
 		(unit 1)
@@
 	)
 	(symbol
+		(lib_name "simbolos-electricos:NPN")
 		(lib_id "simbolos-electricos:NPN")
 		(at 50.8 13.97 0)
